File: pcb/unisolder-mini.kicad_sch (KiCad schematic)
At the start: 0 parts

Commit message: sch: initial port, 80% front pcb
Signed-off-by: Rafael Silva <perigoso@riseup.net>
Parts:
- added BZ1: Buzzer, symbol Device:Buzzer
- added C42, C43, C44, C45, C46, C53, C54, C58, C61, C78, C? (x3): 100n, symbol Device:C_Small
- added C57: 10u, symbol Device:C_Small
- added C60, C62, C? (x2): 10n, symbol Device:C_Small
- added C63, C64, C?: 1n, symbol Device:C_Small
- added D16, D20, D21, D23: BAV99, Package_TO_SOT_SMD:SOT-23, symbol Diode:BAV99
- added D18, D19: D_x2_ACom_KKA, symbol Device:D_x2_ACom_KKA
- added ENCODER, OLED1, OLED2: Header 5, symbol Connector_Generic:Conn_01x05
- added H1, H2, H3, H4: ~, symbol Mechanical:MountingHole_Pad
- added J8: CNTR, symbol Connector_Generic:Conn_01x10
- added J9: PWR, symbol Connector_Generic:Conn_01x06
- added J?: USB_B_Mini, symbol Connector:USB_B_Mini
- added PD1: DEBUG, symbol Connector_Generic:Conn_01x05
- added Q18, Q19, Q21, Q22, Q? (x2): IRLML6401, Package_TO_SOT_SMD:SOT-23, symbol Transistor_FET:IRLML6401
- added R12, R37, R45, R46, R58, R?: 3k, symbol Device:R_Small
- added R23, R32, R70, R? (x5): 1.8k, symbol Device:R_Small
- added R24, R51, R60, R?: 1k, symbol Device:R_Small
- added R25, R26: 27, symbol Device:R_Small
- added R30, R35, R42, R55, R? (x8): 1.5k, symbol Device:R_Small
- added R31, R39: 100, symbol Device:R_Small
- added R38, R48: 47k, symbol Device:R_Small
- added R43, R61, R64: 15k, symbol Device:R_Small
- added R47, R49, R?: 27k, symbol Device:R_Small
- added R?: 10M, symbol Device:R_Small
- added RV2: 2k, symbol Device:R_POT_Small
- added SW1, SW3, SW4: ~, symbol Switch:SW_SPST
- added U12, U13, U18: MCP6V27, symbol unisolder:MCP6V27
- added U14: NP, Package_TO_SOT_THT:TO-92_Inline, symbol Reference_Voltage:LM4041LP-ADJ
- added U4: TC1047AVNB, Package_TO_SOT_SMD:SOT-23, symbol Sensor_Temperature:TC1047AxNB
- added U7: ADUM3160, Package_SO:SOIC-16W_7.5x10.3mm_P1.27mm, symbol Interface_USB:ADUM3160
- added U? (x5): ADG734, Package_SO:TSSOP-20_4.4x6.5mm_P0.65mm, symbol Analog_Switch:ADG734
- added U?: MCP6V28, symbol unisolder:MCP6V28
- added U?: MCP45x1-xxx, symbol unisolder:MCP45x1-xxx
- added U?: REF3030, Package_TO_SOT_SMD:SOT-23, symbol Reference_Voltage:REF3030
- added U?: MCP4651-503, symbol unisolder:MCP46x1-xxx
- added U?: 24LC64, symbol Memory_EEPROM:24LC64
- added U?: MCP47x6, symbol unisolder:MCP47x6
- added Y1: 8MHz, symbol Device:Crystal
- added ZD4: 3.0V, symbol Device:D_Zener
Connections:
- new net: C58.2, R?.1, U14.1 (FB), U14.3 (A), U?.7 (P1A), U?.8 (P0A)
- new net: R?.1, R?.2, U18.1
- new net: R?.1, R?.2, U13.2 (-)
- new net: Q18.3 (D), R30.2, R31.1
- new net: R42.2, R48.2, U13.5 (+)
- new net: R37.2, R38.2, U13.6 (-)
- new net: R38.1, R45.1, U13.7
- new net: C57.2, R32.1
- new net: R26.1, U7.7 (UD+)
- new net: J?.3 (D+), R26.2
- new net: R?.1, R?.2, RV2.3, U18.2 (-)
- new net: C54.1, U7.3 (VDD1), U7.4 (PDEN), U7.5 (SPU)
- new net: U?.12, U?.17, U?.3
- new net: C?.1, R49.1, R60.2, R?.2, U?.2 (-)
- new net: U?.3 (+), U?.6 (P0W)
- new net: C?.2, R55.1, R58.2, R?.1, U?.6
- new net: BZ1.1 (-), R32.2
- new net: Q21.3 (D), R35.2, R39.1
- new net: R?.1, RV2.1, RV2.2
- new net: R?.1, R?.2, R?.2, U18.6 (-)
- new net: R?.1, R?.2, U13.1
- new net: R?.1, R?.2, U13.3 (+)
- new net: R?.1, R?.1, U18.7
- new net: U?.14, U?.19, U?.8
- new net: Q22.1 (G), R?.2, U12.1
- new net: Q22.2 (S), R39.2, U12.2 (-)
- new net: U12.3 (+), U?.9 (P0W)
- new net: D19.3 (A), Q22.3 (D)
- new net: Q19.1 (G), R?.2, U12.7
- new net: D18.3 (A), Q19.3 (D)
- new net: Q19.2 (S), R31.2, U12.6 (-)
- new net: J?.2 (D-), R25.2
- new net: R25.1, U7.6 (UD-)
- new net: U12.5 (+), U?.6 (P1W)
- new net +3V3: C46.1, C58.1, C?.1, D16.2 (A), D18.1 (K), D19.2 (K), D23.2 (A), ENCODER.3 (Pin_3), PD1.2 (Pin_2), Q18.2 (S), Q21.2 (S), R12.1, R24.1, R30.1, R35.1, R?.1, R?.1, SW1.2 (B), SW3.2 (B), SW4.2 (B), U12.8 (V+), U13.8 (V+), U14.2 (K), U18.8 (V+), U4.1 (Vdd), U7.12 (PIN), U7.13 (SPD), U7.14 (VDD2), U7.16 (VBUS2), U?.1 (HVC/A0), U?.1 (IN), U?.10 (P0B), U?.12 (A2), U?.13 (A1), U?.14 (VDD), U?.16 (VDD), U?.3 (VDD), U?.5 (P1B), U?.7 (VDD), U?.8 (VCC), U?.8 (VDD)
- new net -0.6V: J9.4 (Pin_4)
- new net -5V: U13.4 (V-), U18.4 (V-), U?.5 (VSS)
- new net 3.3V: J9.6 (Pin_6)
- new net A1/VDD: OLED1.1 (Pin_1), Q?.3 (D)
- new net A3/VCC: OLED2.5 (Pin_5), Q?.3 (D)
- new net ACH: C63.2, D20.1 (K), D20.2 (A), R61.2, U?.2
- new net B1: ENCODER.5 (Pin_5), R?.2, SW1.1 (A)
- new net B2: ENCODER.4 (Pin_4), R?.2, SW3.1 (A)
- new net B3: ENCODER.2 (Pin_2), R?.2, SW4.1 (A)
- new net BCH: C64.2, D21.1 (K), D21.2 (A), R64.2, U?.9
- new net CBANDA: Q21.1 (G)
- new net CBANDB: Q18.1 (G)
- new net CHPOL: U?.11, U?.20
- new net CHSEL1: U?.1
- new net CHSEL2: U?.10
- new net DGND: J9.2 (Pin_2)
- new net DVdd: J9.3 (Pin_3)
- new net GND: BZ1.2 (+), C42.2, C43.2, C44.2, C45.2, C46.2, C53.2, C54.2, C60.2, C61.1, C62.2, C78.2, C?.2, C?.2, C?.2, C?.2, C?.2, D16.1 (K), D20.3 (K), D21.3 (K), D23.1 (K), ENCODER.1 (Pin_1), J9.1 (Pin_1), J9.5 (Pin_5), OLED1.2 (Pin_2), OLED2.4 (Pin_4), R46.2, R48.1, R51.1, R58.1, R60.1, R?.1, R?.1, R?.1, R?.1, R?.2, R?.2, U12.4 (V-), U4.3 (GND), U7.15 (GND2), U7.9 (GND2), U?.1 (A0), U?.2 (A1), U?.2 (VSS), U?.3 (A2), U?.3 (GND), U?.4 (GND), U?.4 (VSS), U?.4 (VSS), U?.4 (VSS), U?.6 (GND), U?.7 (P0B), U?.7 (WP), ZD4.2 (A)
- new net GND1: J?.5 (GND), R?.2, U7.2 (GND1), U7.8 (GND1)
- new net GNDPWR: H1.1, H2.1, H3.1, H4.1
- new net GNDS: C63.1, C64.1, J8.7 (Pin_7), J8.8 (Pin_8), PD1.3 (Pin_3), R37.1, U?.4, U?.7
- new net HSEL: J8.4 (Pin_4)
- new net ID: J8.3 (Pin_3), R24.2, R70.2
- new net IDIN: C78.1, D23.3 (K), R70.1
- new net IN+: U18.5 (+), U?.13
- new net IN-: U18.3 (+), U?.18
- new net IND1/VDD: Q?.1 (G)
- new net IND3/VCC: Q?.1 (G)
- new net NAP: C45.1, D16.3 (K), R23.1
- new net OLED_CS: OLED2.3 (Pin_3)
- new net OLED_D/C: OLED2.2 (Pin_2)
- new net OLED_RES: OLED2.1 (Pin_1)
- new net OLED_SCK: OLED1.5 (Pin_5)
- new net OLED_SDI: OLED1.4 (Pin_4)
- new net OLED_SDO: OLED1.3 (Pin_3)
- new net ONOFF: J8.6 (Pin_6)
- new net OSC1: C?.1, Y1.1
- new net OSC2: C?.1, Y1.2
- new net PGC: PD1.5 (Pin_5)
- new net PGD: PD1.4 (Pin_4)
- new net SCL: U?.2 (SCL), U?.2 (SCL), U?.5 (SCL), U?.6 (SCL)
- new net SDA: U?.3 (SDA), U?.3 (SDA), U?.4 (SDA), U?.5 (SDA)
- new net SENSEA: D19.1 (K), J8.9 (Pin_9), R61.1
- new net SENSEB: D18.2 (K), J8.10 (Pin_10), R64.1
- new net SHUNT: J8.5 (Pin_5), R42.1
- new net SLEEP: J8.2 (Pin_2), R12.2, R23.2
- new net SPEAKER: C57.1
- new net USBD+: U7.10 (DD+)
- new net USBD-: U7.11 (DD-)
- new net VBUS: C53.1, J?.1 (VBUS), U7.1 (VBUS1)
- new net VDD: Q?.2 (S), Q?.2 (S)
- new net VINT: C60.1, R43.1, R46.1, ZD4.1 (K)
- new net VPP: PD1.1 (Pin_1)
- new net VSHUNT: C?.1, R45.2
- new net Vacdc: C61.2, R47.2, R51.2
- new net Vadc: C62.1, R55.2
- new net Vin: J8.1 (Pin_1), R43.2, R47.1
- new net Voff: R49.2, U?.1 (Vout)
- new net Vref: C42.1, C43.1, C44.1, U?.2 (OUT), U?.6 (VREF)
- new net Vrt: U4.2 (Vout)
- new net Vtemp: C?.1, R?.2, U?.5 (P0A)
- no-connect marks 0 -> 3
Other:
- note added: "Rs1 R37/R42 0.003 1.5K 0.1% 0.004 2.0K 0.1%"
